Commit message: Practical Session 6

File: src/daniel_r2d2/urdf/r2d2.urdf (robot description, URDF)
Before this commit: robot macroed, 5 links, 4 joints
Links:
- removed link lens
- added link left_back_wheel, mass 1; collision cylinder length=0.1 radius=0.035; visual cylinder length=0.1 radius=0.035
- added link left_base, mass 10; collision box size=0.4 0.1 0.1; visual box size=0.4 0.1 0.1
- added link left_front_wheel, mass 1; collision cylinder length=0.1 radius=0.035; visual cylinder length=0.1 radius=0.035
- added link left_gripper, mass 0.05; collision mesh filename=package://urdf_tutorial/meshes/l_finger.dae; visual mesh filename=package://urdf_tutorial/meshes/l_finger.dae
- added link left_leg, mass 10; collision box size=0.6 0.1 0.2; visual box size=0.6 0.1 0.2
- added link left_tip, mass 0.05; collision mesh filename=package://urdf_tutorial/meshes/l_finger_tip.dae; visual mesh filename=package://urdf_tutorial/meshes/l_finger_tip.dae
- added link right_back_wheel, mass 1; collision cylinder length=0.1 radius=0.035; visual cylinder length=0.1 radius=0.035
- added link right_base, mass 10; collision box size=0.4 0.1 0.1; visual box size=0.4 0.1 0.1
- added link right_front_wheel, mass 1; collision cylinder length=0.1 radius=0.035; visual cylinder length=0.1 radius=0.035
- added link right_gripper, mass 0.05; collision mesh filename=package://urdf_tutorial/meshes/l_finger.dae; visual mesh filename=package://urdf_tutorial/meshes/l_finger.dae
- added link right_leg, mass 10; collision box size=0.6 0.1 0.2; visual box size=0.6 0.1 0.2
- added link right_tip, mass 0.05; collision mesh filename=package://urdf_tutorial/meshes/l_finger_tip.dae; visual mesh filename=package://urdf_tutorial/meshes/l_finger_tip.dae
- link base_link: mass None -> 10; geometry collision cylinder length=0.6 radius=0.2; visual cylinder length=0.6 radius=0.2
- link box: mass None -> 1
- link gripper_pole: mass None -> 0.05; geometry collision cylinder length=0.2 radius=0.01; visual cylinder length=0.2 radius=0.01
- link head: mass None -> 2; geometry collision sphere radius=0.2; visual sphere radius=0.2
Joints:
- removed joint lens_joint
- added joint base_to_left_leg: type fixed, parent base_link, child left_leg, origin xyz=0 0.22 0.25
- added joint base_to_right_leg: type fixed, parent base_link, child right_leg, origin xyz=0 -0.22 0.25
- added joint left_back_wheel_joint: type continuous, parent left_base, child left_back_wheel, origin xyz=-0.133333333333 0 -0.085 rpy=0 0 0, axis 0 1 0
- added joint left_base_joint: type fixed, parent left_leg, child left_base, origin xyz=0 0 -0.6
- added joint left_front_wheel_joint: type continuous, parent left_base, child left_front_wheel, origin xyz=0.133333333333 0 -0.085 rpy=0 0 0, axis 0 1 0
- added joint left_gripper_joint: type revolute, parent gripper_pole, child left_gripper, origin xyz=0.2 0.01 0 rpy=0 0 0, axis 0 0 1, limit lower=0.0 upper=0.548 effort=1000.0 velocity=0.5
- added joint left_tip_joint: type fixed, parent left_gripper, child left_tip
- added joint right_back_wheel_joint: type continuous, parent right_base, child right_back_wheel, origin xyz=-0.133333333333 0 -0.085 rpy=0 0 0, axis 0 1 0
- added joint right_base_joint: type fixed, parent right_leg, child right_base, origin xyz=0 0 -0.6
- added joint right_front_wheel_joint: type continuous, parent right_base, child right_front_wheel, origin xyz=0.133333333333 0 -0.085 rpy=0 0 0, axis 0 1 0
- added joint right_gripper_joint: type revolute, parent gripper_pole, child right_gripper, origin xyz=0.2 -0.01 0 rpy=0 0 0, axis 0 0 -1, limit lower=0.0 upper=0.548 effort=1000.0 velocity=0.5
- added joint right_tip_joint: type fixed, parent right_gripper, child right_tip
- joint gripper_extension: limit lower=-${width*2-.02} upper=0 effort=1000.0 velocity=0.5 -> lower=-0.38 upper=0 effort=1000.0 velocity=0.5; origin xyz=${width-.01} 0 0.2 rpy=0 0 0 -> xyz=0.19 0 0.2 rpy=0 0 0
- joint head_swivel: origin xyz=0 0 ${bodylen/2} -> xyz=0 0 0.3
- joint tobox: origin xyz=${.707*width+0.04} 0 ${.707*width} -> xyz=0.1814 0 0.1414
